File: pcb/pcb.kicad_pcb (KiCad board)
At the start: 2 copper layers, 139.8 x 110.8 mm, 114 parts, among them SW1 Switch, SW10 Switch, SW11 Switch, SW12 Switch, SW13 Switch, SW14 Switch, SW15 Switch, SW16 Switch, SW17 Switch, SW18 Switch, SW19 Switch, SW2 Switch, SW20 Switch, SW21 Switch, SW22 Switch, SW23 Switch, SW24 Switch, SW25 Switch, SW26 Switch, SW27 Switch, SW28 Switch, SW29 Switch, SW3 Switch, SW30 Switch, SW31 Switch, SW32 Switch, SW33 Switch, SW34 Switch, SW4 Switch, SW5 Switch, SW6 Switch, SW7 Switch, SW8 Switch, SW9 Switch

Commit message: update to 1.2
Parts:
- removed D35, D36, D37, D38, D39: D, zzkeeb:Diode_1N4148-SOD123
- added D40: D, zzkeeb:Diode_1N4148-SOD123, B.Cu at (30.0, 93.5)
- H1, H2, H3, H4, H5, H6, H7: footprint zzkeeb:Hole_M2 -> zzkeeb:Hole_M2-TH
- MCU1: footprint zzkeeb:MCU_rp2040-zero-smd -> zzkeeb:MCU_rp2040-zero-tht
Connections:
- FiveWay1 pad 1: Net-(D39-A) -> row4
- FiveWay1 pad 2: Net-(D38-A) -> row3
- FiveWay1 pad 3: Net-(D37-A) -> row2
- FiveWay1 pad 5: Net-(D36-A) -> row1
- FiveWay1 pad 6: Net-(D35-A) -> row0
- LED1 pad 1: VCC -> Net-(D40-K)
- LED10 pad 1: VCC -> +5V
- LED11 pad 1: VCC -> +5V
- LED12 pad 1: VCC -> +5V
- LED13 pad 1: VCC -> +5V
- LED14 pad 1: VCC -> +5V
- LED15 pad 1: VCC -> +5V
- LED16 pad 1: VCC -> +5V
- LED17 pad 1: VCC -> +5V
- LED18 pad 1: VCC -> +5V
- LED19 pad 1: VCC -> +5V
- LED2 pad 1: VCC -> +5V
- LED20 pad 1: VCC -> +5V
- LED21 pad 1: VCC -> +5V
- LED22 pad 1: VCC -> +5V
- LED23 pad 1: VCC -> +5V
- LED24 pad 1: VCC -> +5V
- LED25 pad 1: VCC -> +5V
- LED26 pad 1: VCC -> +5V
- LED27 pad 1: VCC -> +5V
- LED28 pad 1: VCC -> +5V
- LED29 pad 1: VCC -> +5V
- LED3 pad 1: VCC -> +5V
- LED30 pad 1: VCC -> +5V
- LED31 pad 1: VCC -> +5V
- LED4 pad 1: VCC -> +5V
- LED5 pad 1: VCC -> +5V
- LED6 pad 1: VCC -> +5V
- LED7 pad 1: VCC -> +5V
- LED8 pad 1: VCC -> +5V
- LED9 pad 1: VCC -> +5V
- MCU1 pad 21: VCC -> unconnected-(MCU1-3V3-Pad21)
- MCU1 pad 23: unconnected-(MCU1-5V-Pad23) -> +5V
Routing:
- net +5V: track 0.00 -> 851.2 mm, vias 0 -> 31
- net VCC: track 845.8 -> 0.00 mm, vias 31 -> 0
- net GND: track 0.00 -> 22.6 mm, vias 4 -> 1
- net Net-(D37-A): track 22.3 -> 0.00 mm
- net Net-(D38-A): track 14.9 -> 0.00 mm, vias 1 -> 0
- net Net-(D35-A): track 13.4 -> 0.00 mm
- net Net-(D36-A): track 13.3 -> 0.00 mm
- net row3: track 210.4 -> 222.9 mm, vias 1 -> 2
- net Net-(D39-A): track 4.39 -> 0.00 mm
- net row1: track 223.9 -> 228.0 mm
- net row2: track 252.7 -> 248.7 mm
- net Net-(D40-K): track 0.00 -> 3.40 mm
- net row4: track 248.7 -> 251.9 mm
- net col5: track 191.2 -> 188.2 mm, vias 7 -> 6
- net col6: track 216.1 -> 213.2 mm, vias 7 -> 6
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Other:
- outline, holes or cut-outs redrawn
- board text added: "KeyGameBoard v1.2"
- board text removed: "KeyGameBoard v1.1"
