File: pcb/pcb.kicad_sch (KiCad schematic)
At the start: 113 parts, among them SW1 Switch, SW10 Switch, SW11 Switch, SW12 Switch, SW13 Switch, SW14 Switch, SW15 Switch, SW16 Switch, SW17 Switch, SW18 Switch, SW19 Switch, SW2 Switch, SW20 Switch, SW21 Switch, SW22 Switch, SW23 Switch, SW24 Switch, SW25 Switch, SW26 Switch, SW27 Switch, SW28 Switch, SW29 Switch, SW3 Switch, SW30 Switch, SW31 Switch, SW32 Switch, SW33 Switch, SW34 Switch, SW4 Switch, SW5 Switch, SW6 Switch, SW7 Switch, SW8 Switch, SW9 Switch

Commit message: update to 1.2
Parts:
- removed D35, D36, D37, D38, D39: D, zzkeeb:Diode_1N4148-SOD123, symbol zzkeeb:Diode
- added D40: D, zzkeeb:Diode_1N4148-SOD123, symbol Device:D
- H1, H2, H3, H4, H5, H6, H7: footprint zzkeeb:Hole_M2 -> zzkeeb:Hole_M2-TH
- MCU1: footprint zzkeeb:MCU_rp2040-zero-smd -> zzkeeb:MCU_rp2040-zero-tht
Connections:
- net row0: now also FiveWay1.6
- net row1: now also FiveWay1.5
- net row2: now also FiveWay1.3
- net row3: now also FiveWay1.2
- net row4: now also FiveWay1.1
- net +5V: now reaches MCU1.23 (5V)
- net +5V: now also LED10.1 (VDD), LED11.1 (VDD), LED12.1 (VDD), LED13.1 (VDD), LED14.1 (VDD), LED15.1 (VDD), LED16.1 (VDD), LED17.1 (VDD), LED18.1 (VDD), LED19.1 (VDD), LED2.1 (VDD), LED20.1 (VDD), LED21.1 (VDD), LED22.1 (VDD), LED23.1 (VDD), LED24.1 (VDD), LED25.1 (VDD), LED26.1 (VDD), LED27.1 (VDD), LED28.1 (VDD), LED29.1 (VDD), LED3.1 (VDD), LED30.1 (VDD), LED31.1 (VDD), LED4.1 (VDD), LED5.1 (VDD), LED6.1 (VDD), LED7.1 (VDD), LED8.1 (VDD), LED9.1 (VDD), D40.2 (A)
- removed net VCC: LED1.1 (VDD), LED10.1 (VDD), LED11.1 (VDD), LED12.1 (VDD), LED13.1 (VDD), LED14.1 (VDD), LED15.1 (VDD), LED16.1 (VDD), LED17.1 (VDD), LED18.1 (VDD), LED19.1 (VDD), LED2.1 (VDD), LED20.1 (VDD), LED21.1 (VDD), LED22.1 (VDD), LED23.1 (VDD), LED24.1 (VDD), LED25.1 (VDD), LED26.1 (VDD), LED27.1 (VDD), LED28.1 (VDD), LED29.1 (VDD), LED3.1 (VDD), LED30.1 (VDD), LED31.1 (VDD), LED4.1 (VDD), LED5.1 (VDD), LED6.1 (VDD), LED7.1 (VDD), LED8.1 (VDD), LED9.1 (VDD), MCU1.21 (3V3)
- new net: D40.1 (K), LED1.1 (VDD)
